Commit message: navigation param error

File: src/my_kwj_urdf/urdf.urdf (robot description, URDF)
Before this commit: robot KWJBot, 2 links, 1 joints
Links:
- removed link wheel_link
- added link left_wheel, mass 0.1; collision cylinder length=0.01 radius=0.05; visual cylinder length=0.05 radius=0.1
- added link right_wheel, mass 0.1; collision cylinder length=0.01 radius=0.05; visual cylinder length=0.05 radius=0.1
- link base_link: mass None -> 1; geometry visual box size=0.5 0.5 0.1
Joints:
- removed joint base_joint
- added joint left_wheel_joint: type continuous, parent base_link, child left_wheel, origin xyz=-0.25 0.0 0.0 rpy=0 0 0
- added joint right_wheel_joint: type continuous, parent base_link, child right_wheel, origin xyz=0.25 0.0 0.0 rpy=0 0 0

Commit message: not move

File: src/my_kwj_urdf/urdf.urdf (robot description, URDF)
Before this commit: robot KWJBot, 3 links, 2 joints
Links:
- added link base_footprint
- link base_link: geometry visual box size=0.2 0.2 0.13
- link left_wheel: geometry collision cylinder length=0.01 radius=0.03; visual cylinder length=0.01 radius=0.015
- link right_wheel: geometry collision cylinder length=0.01 radius=0.03; visual cylinder length=0.01 radius=0.015
Joints:
- added joint base_joint: type fixed, parent base_footprint, child base_link
- joint left_wheel_joint: axis (none) -> 1 0 0; origin xyz=-0.25 0.0 0.0 rpy=0 0 0 -> xyz=-0.0 0.0 0.0 rpy=0 0 0
- joint right_wheel_joint: axis (none) -> 1 0 0; origin xyz=0.25 0.0 0.0 rpy=0 0 0 -> xyz=0.0 0.0 0.0 rpy=0 0 0

Commit message: success navigation

File: src/my_kwj_urdf/urdf.urdf (robot description, URDF)
Before this commit: robot KWJBot, 4 links, 3 joints
Links:
- removed link base_footprint
- added link odom
Joints:
- joint base_joint: parent base_footprint -> odom
